File: gsm-iot-core.sch (KiCad schematic (older format))
At the start: 95 parts, among them J1 MICRO_SD_HINGE - Micro SD soc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, P1 CONN_01X02, P2 CONN_01X04, P3 CONN_01X15, P4 CONN_01X17, P5 CONN_01X01, P6 CONN_01X01, P7 CONN_01X01, P8 CONN_01X01, P9 Chip anten, Q1 2SC1815, Q2 2SC1815, SW1 SW_PUSH, SW2 SW_PUSH, U1 STM32F405RGTx, U2 MP2365DN, U3 LP2985-50DBVR, U4 MMA7660, U5 SIM800C, U6 SIM HOLD - PPSS-6P, Y1 8MHz, Y2 32.768MHz

Commit message: branch upstream
Parts:
- added C?: 100nF, symbol C_Small
Connections:
- net GND: now also C?.2
- net PB3_BUTTON: now also C?.1
Other:
- moved on the sheet: R13, SW2
Changed lines of the file:
@@
 L SW_PUSH SW2
 U 1 1 57B13478
-P 10215 8585
-F 0 "SW2" H 10215 8840 50  0000 C CNN
-F 1 "SW_PUSH" H 10215 8749 50  0000 C CNN
-F 2 "button:SW_SPST_B3U-1000P" H 10215 8585 50  0001 C CNN
-F 3 "" H 10215 8585 50  0000 C CNN
-	1    10215 8585
+P 10350 8600
+F 0 "SW2" H 10350 8855 50  0000 C CNN
+F 1 "SW_PUSH" H 10350 8764 50  0000 C CNN
+F 2 "button:SW_SPST_B3U-1000P" H 10350 8600 50  0001 C CNN
+F 3 "" H 10350 8600 50  0000 C CNN
+	1    10350 8600
 	0    1    1    0
 $EndComp
@@
 L GND #PWR017
 U 1 1 57B13C12
-P 10215 8885
-F 0 "#PWR017" H 10215 8635 50  0001 C CNN
-F 1 "GND" H 10220 8712 50  0000 C CNN
-F 2 "" H 10215 8885 50  0000 C CNN
-F 3 "" H 10215 8885 50  0000 C CNN
-	1    10215 8885
+P 10350 9000
+F 0 "#PWR017" H 10350 8750 50  0001 C CNN
+F 1 "GND" H 10355 8827 50  0000 C CNN
+F 2 "" H 10350 9000 50  0000 C CNN
+F 3 "" H 10350 9000 50  0000 C CNN
+	1    10350 9000
 	1    0    0    -1
 $EndComp
@@
 L R_Small R13
 U 1 1 57B13D2A
-P 10215 8185
-F 0 "R13" V 10115 8185 50  0000 C CNN
-F 1 "10K" V 10215 8185 50  0000 C CNN
-F 2 "Resistors_SMD:R_0603" H 10215 8185 50  0001 C CNN
-F 3 "" H 10215 8185 50  0000 C CNN
-	1    10215 8185
+P 10350 8100
+F 0 "R13" V 10250 8100 50  0000 C CNN
+F 1 "10K" V 10365 8115 50  0000 C CNN
+F 2 "Resistors_SMD:R_0603" H 10350 8100 50  0001 C CNN
+F 3 "" H 10350 8100 50  0000 C CNN
+	1    10350 8100
 	-1   0    0    1
 $EndComp
-Text GLabel 10055 8350 0    79   Input ~ 16
-PB3_BUTTON
 $Comp
 L Led_Small D4
@@
 L +3.3V #PWR049
 U 1 1 57ADA0C5
-P 10215 8085
-F 0 "#PWR049" H 10215 7935 50  0001 C CNN
-F 1 "+3.3V" H 10230 8258 50  0000 C CNN
-F 2 "" H 10215 8085 50  0000 C CNN
-F 3 "" H 10215 8085 50  0000 C CNN
-	1    10215 8085
+P 10350 7900
+F 0 "#PWR049" H 10350 7750 50  0001 C CNN
+F 1 "+3.3V" H 10365 8073 50  0000 C CNN
+F 2 "" H 10350 7900 50  0000 C CNN
+F 3 "" H 10350 7900 50  0000 C CNN
+	1    10350 7900
 	1    0    0    -1
 $EndComp
@@
 	20825 4700 20825 4900
 Wire Wire Line
-	10215 8285 10055 8285
-Wire Wire Line
-	10055 8285 10055 8350
-Wire Wire Line
 	19880 3130 19920 3130
 Wire Wire Line
@@
 Wire Wire Line
 	16300 9050 16300 8950
+Text GLabel 10600 8250 2    79   Input ~ 16
+PB3_BUTTON
+Wire Wire Line
+	10350 8900 10350 9000
+Wire Wire Line
+	10350 8200 10350 8300
+Wire Wire Line
+	10350 7900 10350 8000
+$Comp
+L C_Small C?
+U 1 1 57DA5C17
+P 9950 8600
+F 0 "C?" H 10042 8646 50  0000 L CNN
+F 1 "100nF" H 10042 8555 50  0000 L CNN
+F 2 "" H 9950 8600 50  0000 C CNN
+F 3 "" H 9950 8600 50  0000 C CNN
+	1    9950 8600
+	1    0    0    -1
+$EndComp
+Wire Wire Line
+	9950 8500 9950 8250
+Wire Wire Line
+	9950 8250 10600 8250
+Connection ~ 10350 8250
+Wire Wire Line
+	9950 8700 9950 8950
+Wire Wire Line
+	9950 8950 10350 8950
+Connection ~ 10350 8950
 $EndSCHEMATC
