File: gsm-iot-core.sch (KiCad schematic (older format))
At the start: 90 parts, among them J1 MICRO_SD_HINGE - Micro SD soc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, P1 CONN_01X16, P2 CONN_01X04, P3 CONN_01X16, P5 Chip anten, Q1 2SC1815, Q2 2SC1815, SW1 SW_PUSH, SW3 SW_PUSH, U1 MP2365DN, U2 LP2985-50DBVR, U3 STM32F405RGTx, U4 MMA7660, U5 SIM800C, U6 SIM HOLD - PPSS-6P, X1 CRYSTAL-24M, Y3 32.768MHz

Commit message: update
Parts:
- removed P1, P3: CONN_01X16, Pin_Headers:Pin_Header_Straight_1x16, symbol CONN_01X16
- removed P2: CONN_01X04, Pin_Headers:Pin_Header_Straight_1x04, symbol CONN_01X04
- added P1, P2: CONN_01X18, Pin_Headers:Pin_Header_Straight_1x18, symbol CONN_01X18
Changed lines of the file:
@@
 NoConn ~ 17740 2590
 NoConn ~ 19250 5150
-$Comp
-L CONN_01X04 P2
-U 1 1 57DA6BB0
-P 14025 2840
-F 0 "P2" H 14103 2881 50  0000 L CNN
-F 1 "CONN_01X04" H 14103 2790 50  0000 L CNN
-F 2 "Pin_Headers:Pin_Header_Straight_1x04" H 14025 2840 50  0001 C CNN
-F 3 "" H 14025 2840 50  0000 C CNN
-	1    14025 2840
-	1    0    0    -1
-$EndComp
-Text GLabel 13825 2990 0    60   Input Italic 0
+Text GLabel 15300 9000 0    60   Input Italic 0
 PA13_SWDIO
-Text GLabel 13825 2890 0    60   Input Italic 0
+Text GLabel 15300 8900 0    60   Input Italic 0
 PA14_SWCLK
-$Comp
-L GND #PWR052
-U 1 1 57DA6BB1
-P 13825 2790
-F 0 "#PWR052" H 13825 2540 50  0001 C CNN
-F 1 "GND" V 13830 2662 50  0000 R CNN
-F 2 "" H 13825 2790 50  0000 C CNN
-F 3 "" H 13825 2790 50  0000 C CNN
-	1    13825 2790
-	0    1    1    0
-$EndComp
-$Comp
-L +3.3V #PWR053
-U 1 1 57DA6BB2
-P 13825 2690
-F 0 "#PWR053" H 13825 2540 50  0001 C CNN
-F 1 "+3.3V" H 13840 2863 50  0000 C CNN
-F 2 "" H 13825 2690 50  0000 C CNN
-F 3 "" H 13825 2690 50  0000 C CNN
-	1    13825 2690
-	1    0    0    -1
-$EndComp
 $Comp
 L SMF05C D6
@@
 $EndComp
 $Comp
-L GND #PWR054
+L GND #PWR052
 U 1 1 57DA6BB4
 P 19400 5000
-F 0 "#PWR054" H 19400 4750 50  0001 C CNN
+F 0 "#PWR052" H 19400 4750 50  0001 C CNN
 F 1 "GND" H 19405 4827 50  0000 C CNN
 F 2 "" H 19400 5000 50  0000 C CNN
@@
 NoConn ~ 19100 5525
 $Comp
-L GND #PWR055
+L GND #PWR053
 U 1 1 57DA6BB5
 P 18900 6125
-F 0 "#PWR055" H 18900 5875 50  0001 C CNN
+F 0 "#PWR053" H 18900 5875 50  0001 C CNN
 F 1 "GND" H 18905 5952 50  0000 C CNN
 F 2 "" H 18900 6125 50  0000 C CNN
@@
 $EndComp
 $Comp
-L GND #PWR056
+L GND #PWR054
 U 1 1 57DA6BB8
 P 19560 5560
-F 0 "#PWR056" H 19560 5310 50  0001 C CNN
+F 0 "#PWR054" H 19560 5310 50  0001 C CNN
 F 1 "GND" H 19565 5387 50  0000 C CNN
 F 2 "" H 19560 5560 50  0000 C CNN
@@
 RST
 $Comp
-L +3.3V #PWR057
+L +3.3V #PWR055
 U 1 1 57DA6BB9
 P 10350 7900
-F 0 "#PWR057" H 10350 7750 50  0001 C CNN
+F 0 "#PWR055" H 10350 7750 50  0001 C CNN
 F 1 "+3.3V" H 10365 8073 50  0000 C CNN
 F 2 "" H 10350 7900 50  0000 C CNN
@@
 Text GLabel 11700 5400 2    60   Input ~ 0
 PB10
-Text GLabel 15300 8600 0    60   Input ~ 0
+Text GLabel 15300 8500 0    60   Input ~ 0
 PC13
-Text GLabel 15300 8500 0    60   Input ~ 0
+Text GLabel 15300 8400 0    60   Input ~ 0
 PC0
-Text GLabel 15300 8400 0    60   Input ~ 0
+Text GLabel 15300 8300 0    60   Input ~ 0
 PC1
-Text GLabel 15300 8300 0    60   Input ~ 0
+Text GLabel 15300 8200 0    60   Input ~ 0
 PC2
-Text GLabel 15300 8200 0    60   Input ~ 0
+Text GLabel 15300 8100 0    60   Input ~ 0
 PC3
-Text GLabel 15300 8100 0    60   Input ~ 0
+Text GLabel 15300 8000 0    60   Input ~ 0
 PA0
-Text GLabel 15300 8000 0    60   Input ~ 0
+Text GLabel 15300 7900 0    60   Input ~ 0
 PA1
-Text GLabel 15300 7900 0    60   Input ~ 0
+Text GLabel 15300 7800 0    60   Input ~ 0
 PA2
 Text GLabel 16500 7800 0    60   Input ~ 0
 PA3
 $Comp
-L +3.3V #PWR058
+L +3.3V #PWR056
 U 1 1 57DA6BBF
 P 16450 7600
-F 0 "#PWR058" H 16450 7450 50  0001 C CNN
+F 0 "#PWR056" H 16450 7450 50  0001 C CNN
 F 1 "+3.3V" H 16465 7773 50  0000 C CNN
 F 2 "" H 16450 7600 50  0000 C CNN
@@
 $EndComp
 $Comp
-L GND #PWR059
+L GND #PWR057
 U 1 1 57DA6BC0
-P 14950 7800
-F 0 "#PWR059" H 14950 7550 50  0001 C CNN
-F 1 "GND" V 14955 7672 50  0000 R CNN
-F 2 "" H 14950 7800 50  0000 C CNN
-F 3 "" H 14950 7800 50  0000 C CNN
-	1    14950 7800
-	1    0    0    -1
-$EndComp
-$Comp
-L GND #PWR060
+P 14700 7700
+F 0 "#PWR057" H 14700 7450 50  0001 C CNN
+F 1 "GND" V 14705 7572 50  0000 R CNN
+F 2 "" H 14700 7700 50  0000 C CNN
+F 3 "" H 14700 7700 50  0000 C CNN
+	1    14700 7700
+	1    0    0    -1
+$EndComp
+$Comp
+L GND #PWR058
 U 1 1 57DA6BC2
-P 15000 9150
-F 0 "#PWR060" H 15000 8900 50  0001 C CNN
-F 1 "GND" V 15005 9022 50  0000 R CNN
-F 2 "" H 15000 9150 50  0000 C CNN
-F 3 "" H 15000 9150 50  0000 C CNN
-	1    15000 9150
+P 15000 9250
+F 0 "#PWR058" H 15000 9000 50  0001 C CNN
+F 1 "GND" V 15005 9122 50  0000 R CNN
+F 2 "" H 15000 9250 50  0000 C CNN
+F 3 "" H 15000 9250 50  0000 C CNN
+	1    15000 9250
 	1    0    0    -1
 $EndComp
@@
 PA6
 $Comp
-L GND #PWR061
+L GND #PWR059
 U 1 1 57DA6BC3
 P 16100 7700
-F 0 "#PWR061" H 16100 7450 50  0001 C CNN
+F 0 "#PWR059" H 16100 7450 50  0001 C CNN
 F 1 "GND" V 16105 7572 50  0000 R CNN
 F 2 "" H 16100 7700 50  0000 C CNN
@@
 $EndComp
 $Comp
-L +3.3V #PWR062
+L +3.3V #PWR060
 U 1 1 57DA6BC4
-P 16450 9100
-F 0 "#PWR062" H 16450 8950 50  0001 C CNN
-F 1 "+3.3V" H 16300 9250 50  0000 L CNN
-F 2 "" H 16450 9100 50  0000 C CNN
-F 3 "" H 16450 9100 50  0000 C CNN
-	1    16450 9100
+P 16450 9300
+F 0 "#PWR060" H 16450 9150 50  0001 C CNN
+F 1 "+3.3V" H 16300 9450 50  0000 L CNN
+F 2 "" H 16450 9300 50  0000 C CNN
+F 3 "" H 16450 9300 50  0000 C CNN
+	1    16450 9300
 	0    -1   -1   0
 $EndComp
@@
 Text GLabel 16500 8900 0    60   Input ~ 0
 PB15
-Text GLabel 15300 8900 0    60   Input ~ 0
+Text GLabel 15300 8800 0    60   Input ~ 0
 PB4
-Text GLabel 15300 8800 0    60   Input ~ 0
+Text GLabel 15300 8700 0    60   Input ~ 0
 PB8
-Text GLabel 15300 8700 0    60   Input ~ 0
+Text GLabel 15300 8600 0    60   Input ~ 0
 PB9
-Text GLabel 15250 7600 0    60   Input ~ 0
+Text GLabel 15250 7500 0    60   Input ~ 0
 VBAT
 $Comp
-L GND #PWR063
+L GND #PWR061
 U 1 1 57DA6BC5
-P 16200 9150
-F 0 "#PWR063" H 16200 8900 50  0001 C CNN
-F 1 "GND" V 16205 9022 50  0000 R CNN
-F 2 "" H 16200 9150 50  0000 C CNN
-F 3 "" H 16200 9150 50  0000 C CNN
-	1    16200 9150
+P 16200 9350
+F 0 "#PWR061" H 16200 9100 50  0001 C CNN
+F 1 "GND" V 16205 9222 50  0000 R CNN
+F 2 "" H 16200 9350 50  0000 C CNN
+F 3 "" H 16200 9350 50  0000 C CNN
+	1    16200 9350
 	1    0    0    -1
 $EndComp
@@
 $EndComp
 $Comp
-L GND #PWR064
+L GND #PWR062
 U 1 1 57DC1DA6
 P 800 4500
-F 0 "#PWR064" H 800 4250 50  0001 C CNN
+F 0 "#PWR062" H 800 4250 50  0001 C CNN
 F 1 "GND" H 805 4327 50  0000 C CNN
 F 2 "" H 800 4500 50  0000 C CNN
@@
 $EndComp
 $Comp
-L +5V #PWR065
-U 1 1 57EB7FE1
-P 15250 9100
-F 0 "#PWR065" H 15250 8950 50  0001 C CNN
-F 1 "+5V" H 15265 9273 50  0000 C CNN
-F 2 "" H 15250 9100 50  0000 C CNN
-F 3 "" H 15250 9100 50  0000 C CNN
-	1    15250 9100
-	0    -1   -1   0
-$EndComp
-$Comp
-L GND #PWR066
+L GND #PWR064
 U 1 1 57EDC919
 P 8850 10450
-F 0 "#PWR066" H 8850 10200 50  0001 C CNN
+F 0 "#PWR064" H 8850 10200 50  0001 C CNN
 F 1 "GND" H 8855 10277 50  0000 C CNN
 F 2 "" H 8850 10450 50  0000 C CNN
@@
 	2000 13300 1600 13300
 $Comp
-L +3.3V #PWR067
+L +3.3V #PWR065
 U 1 1 57EE83AC
 P 7700 9850
-F 0 "#PWR067" H 7700 9700 50  0001 C CNN
+F 0 "#PWR065" H 7700 9700 50  0001 C CNN
 F 1 "+3.3V" H 7715 10023 50  0000 C CNN
 F 2 "" H 7700 9850 50  0000 C CNN
@@
 	12350 4400 12500 4400
 $Comp
-L GND #PWR068
+L GND #PWR066
 U 1 1 57EEDEDB
 P 12500 4650
-F 0 "#PWR068" H 12500 4400 50  0001 C CNN
+F 0 "#PWR066" H 12500 4400 50  0001 C CNN
 F 1 "GND" H 12505 4477 50  0000 C CNN
 F 2 "" H 12500 4650 50  0000 C CNN
@@
 Text GLabel 16500 8300 0    60   Input ~ 0
 PB2
-$Comp
-L CONN_01X16 P1
-U 1 1 57F16AB1
+Wire Wire Line
+	15000 9100 15000 9250
+Wire Wire Line
+	16500 7700 16100 7700
+Wire Wire Line
+	16500 7600 16450 7600
+Wire Wire Line
+	16500 9200 16200 9200
+Wire Wire Line
+	16200 9200 16200 9350
+$Comp
+L +3.3V #PWR067
+U 1 1 57F1FC6A
+P 14850 7600
+F 0 "#PWR067" H 14850 7450 50  0001 C CNN
+F 1 "+3.3V" H 14865 7773 50  0000 C CNN
+F 2 "" H 14850 7600 50  0000 C CNN
+F 3 "" H 14850 7600 50  0000 C CNN
+	1    14850 7600
+	1    0    0    -1
+$EndComp
+Wire Wire Line
+	16500 9300 16450 9300
+$Comp
+L CONN_01X18 P2
+U 1 1 57F1F53E
+P 16700 8450
+F 0 "P2" H 16778 8491 50  0000 L CNN
+F 1 "CONN_01X18" H 16778 8400 50  0000 L CNN
+F 2 "Pin_Headers:Pin_Header_Straight_1x18" H 16700 8450 50  0001 C CNN
+F 3 "" H 16700 8450 50  0000 C CNN
+	1    16700 8450
+	1    0    0    -1
+$EndComp
+$Comp
+L CONN_01X18 P1
+U 1 1 57F2125F
 P 15500 8350
 F 0 "P1" H 15578 8391 50  0000 L CNN
-F 1 "CONN_01X16" H 15578 8300 50  0000 L CNN
-F 2 "Pin_Headers:Pin_Header_Straight_1x16" H 15500 8350 50  0001 C CNN
+F 1 "CONN_01X18" H 15578 8300 50  0000 L CNN
+F 2 "Pin_Headers:Pin_Header_Straight_1x18" H 15500 8350 50  0001 C CNN
 F 3 "" H 15500 8350 50  0000 C CNN
 	1    15500 8350
 	1    0    0    -1
 $EndComp
-$Comp
-L CONN_01X16 P3
-U 1 1 57F16E31
-P 16700 8350
-F 0 "P3" H 16778 8391 50  0000 L CNN
-F 1 "CONN_01X16" H 16778 8300 50  0000 L CNN
-F 2 "Pin_Headers:Pin_Header_Straight_1x16" H 16700 8350 50  0001 C CNN
-F 3 "" H 16700 8350 50  0000 C CNN
-	1    16700 8350
-	1    0    0    -1
-$EndComp
-Wire Wire Line
-	15300 7600 15250 7600
-Wire Wire Line
-	15000 9000 15300 9000
-Wire Wire Line
-	15300 9100 15250 9100
-Wire Wire Line
-	15000 9000 15000 9150
-Wire Wire Line
-	16500 7700 16100 7700
-Wire Wire Line
-	16500 7600 16450 7600
-Wire Wire Line
-	16500 9000 16200 9000
-Wire Wire Line
-	16200 9000 16200 9150
-Wire Wire Line
-	14950 7800 15300 7800
-$Comp
-L +3.3V #PWR069
-U 1 1 57F1FC6A
-P 14800 7700
-F 0 "#PWR069" H 14800 7550 50  0001 C CNN
-F 1 "+3.3V" H 14815 7873 50  0000 C CNN
-F 2 "" H 14800 7700 50  0000 C CNN
-F 3 "" H 14800 7700 50  0000 C CNN
-	1    14800 7700
-	1    0    0    -1
-$EndComp
-Wire Wire Line
-	15300 7700 14800 7700
-Wire Wire Line
-	16500 9100 16450 9100
+Wire Wire Line
+	15250 7500 15300 7500
+Wire Wire Line
+	15250 9200 15300 9200
+Wire Wire Line
+	15300 7600 14850 7600
+$Comp
+L +5V #PWR063
+U 1 1 57EB7FE1
+P 15250 9200
+F 0 "#PWR063" H 15250 9050 50  0001 C CNN
+F 1 "+5V" H 15265 9373 50  0000 C CNN
+F 2 "" H 15250 9200 50  0000 C CNN
+F 3 "" H 15250 9200 50  0000 C CNN
+	1    15250 9200
+	0    -1   -1   0
+$EndComp
+Wire Wire Line
+	15300 9100 15000 9100
+Wire Wire Line
+	15300 7700 14700 7700
 $EndSCHEMATC

Commit message: Fix power part of schematic & footprint crystal
Parts:
- removed C24: 22uF, lib:C_0603, symbol C_Small
- added C15: 10nF, lib:C_0603, symbol C_Small
- C13: renamed from C22; value 22uF -> 47uF
- L1: value 3.3uH-3.2A -> 4.7uH-2.2A; footprint Choke_SMD:Choke_SMD_Wuerth-WE-PD2-Typ-MS -> Choke_SMD:Choke_SMD_6.3x6.3_H3
- R8: renamed from R11; value 7.5k-1% -> 10k-1%
- R9: renamed from R12; value 25.5k-1% -> 33,6k-1%
- renumbered C12 to C1, C20 to C10, C15 to C11, C21 to C12, C23 to C14, C1 to C16, C25 to C17, C2 to C18, C3 to C19, C29 to C2, C4 to C20, C5 to C21, C26 to C22, C27 to C23, C6 to C24, C7 to C25, C28 to C26, C34 to C27, C35 to C28, C36 to C29, C8 to C3, C37 to C30, C38 to C31, C39 to C32, C40 to C33, C41 to C34, C17 to C4, C18 to C5, C13 to C6, C10 to C7, C11 to C8, C14 to C9, D3 to D2, D4 to D3, D5 to D4, D6 to D5, D7 to D6, D8 to D7, P5 to P3, Q2 to Q1, Q1 to Q2, R4 to R1, R13 to R10, R14 to R11, R15 to R12, R16 to R13, R17 to R14, R1 to R15, R18 to R16, R20 to R17, R22 to R18, R23 to R19, R5 to R2, R24 to R20, R25 to R21, R26 to R22, R27 to R23, R30 to R24, R28 to R25, R29 to R26, R32 to R27, R31 to R28, R33 to R29, R6 to R3, R7 to R4, R8 to R5, R9 to R6, R10 to R7, SW3 to SW2, Y3 to Y1
Connections:
- net GND: now also C15.2; no longer U2.4 (BYPASS)
- net PA0: now also P1.9 (P9); no longer P1.6 (P6)
- net PA1: now also P1.10 (P10); no longer P1.5 (P5)
- net PA13_SWDIO: no longer P1.16 (P16)
- net PA14_SWCLK: no longer P1.15 (P15)
- net PA2: now also P1.11 (P11); no longer P1.4 (P4)
- net PA3: now also P1.12 (P12); no longer P2.3 (P3)
- net PA4: now also P1.13 (P13); no longer P2.4 (P4)
- net PA5: now also P1.14 (P14); no longer P2.5 (P5)
- net PA6: now also P1.15 (P15); no longer P2.6 (P6)
- net PB1: now also P1.16 (P16); no longer P2.7 (P7)
- net PB10: no longer P2.9 (P9)
- net PB11: no longer P2.10 (P10)
- net PB12: no longer P2.11 (P11)
- net PB13: no longer P2.12 (P12)
- net PB14: no longer P2.13 (P13)
- net PB15: no longer P2.14 (P14)
- net PB2: no longer P2.8 (P8)
- net PB4: no longer P1.14 (P14)
- net PB8: no longer P1.13 (P13)
- net PB9: no longer P1.12 (P12)
- net PC0: now also P1.5 (P5); no longer P1.10 (P10)
- net PC1: now also P1.6 (P6); no longer P1.9 (P9)
- net PC13: now also P1.4 (P4); no longer P1.11 (P11)
- net PC2: now also P1.7 (P7); no longer P1.8 (P8)
- net PC3: now also P1.8 (P8); no longer P1.7 (P7)
- net VDD: now also C13.1, R9.1
- new net: C15.1, U2.4 (BYPASS)
Other:
- moved on the sheet: C13, D2, D3, L1, R10, R8, R9

Commit message: Modify microSD diagram & connect betwenn MMA7660 and STM
Parts:
- removed P1, P2: CONN_01X18, Pin_Headers:Pin_Header_Straight_1x18, symbol CONN_01X18
- added P1, P2: CONN_01X17, Pin_Headers:Pin_Header_Straight_1x17, symbol CONN_01X17
- added R30, R31, R32, R33: 47K, lib:R_0603, symbol R_Small
- C8: value 0.2uF -> 2.2uF
- R11: value 10M -> 47K
- X1: footprint lib:Crystal_SMD_5032_4Pads -> lib:Crystal_SMD_3225_4Pads
Connections:
- net PA2 is gone; now on net SIM800C_RXD: U3.16 (ADC1_IN2/ADC2_IN2/ADC3_IN2/TIM2_CH3/TIM5_CH3/TIM9_CH1/USART2_TX/PA2)
- net PA3 is gone; now on net SIM800C_TXD: U3.17 (ADC1_IN3/ADC2_IN3/ADC3_IN3/TIM2_CH4/TIM5_CH4/TIM9_CH2/USART2_RX/USB_OTG_HS_ULPI_D0/PA3)
- net +3V3: now also R11.2, P1.1 (P1), P1.17 (P17), P2.1 (P1), R30.2, R31.2, R32.2, R33.2
- net +5V: now also P2.17 (P17)
- net GND: now also P1.16 (P16), P1.2 (P2), P2.16 (P16), P2.2 (P2); no longer R11.2
- net PA0: now also P2.3 (P3)
- net PA1: now also P1.3 (P3)
- net PA13_SWDIO: now also P1.14 (P14)
- net PA14_SWCLK: now also P1.15 (P15)
- net PA4: now also P1.4 (P4)
- net PA5: now also P1.5 (P5)
- net PA6: now also P1.6 (P6)
- net PB1: now also U4.5 (INT)
- net PB12: now also P1.7 (P7)
- net PB13: now also P1.8 (P8)
- net PB14: now also P1.9 (P9)
- net PB15: now also P1.10 (P10)
- net PB4: now also P2.15 (P15)
- net PB5: now also P2.14 (P14); no longer U4.5 (INT)
- net PB8: now also P2.11 (P11)
- net PB9: now also P2.10 (P10)
- net PC0: now also P2.7 (P7)
- net PC1: now also P2.6 (P6)
- net PC10_SDIO_D2: now also R11.1
- net PC11_SDIO_D3: now also R30.1; no longer R11.1
- net PC13: now also P2.8 (P8)
- net PC2: now also P2.5 (P5)
- net PC3: now also P2.4 (P4)
- net PC8_SDIO_D0: now also R32.1
- net PC9_SDIO_D1: now also R33.1
- net PD2_SDIO_CMD: now also R31.1
- net SIM800C_RXD: no longer U3.37 (PC6/I2S2_MCK/SDIO_D6/TIM3_CH1/TIM8_CH1/USART6_TX)
- net SIM800C_TXD: no longer U3.38 (PC7/I2S3_MCK/SDIO_D7/TIM3_CH2/TIM8_CH2/USART6_RX)
- net SIM800C_VDD: no longer C28.1, D5.6
- net VBAT: now also P2.9 (P9)
- net PA8_SDIO_SW: no longer names the net of J1.9 (GND1)
- net PA8_SDIO_SW: no longer U3.41 (I2C3_SCL/RCC_MCO_1/TIM1_CH1/USART1_CK/USB_OTG_FS_SOF/PA8)
- net PB10 renamed PB10_SCL
- net PB10_SCL: now also R16.2, U4.6 (SCL)
- net PB11 renamed PB11_SDA
- net PB11_SDA: now also R17.2, U4.7 (SDA)
- net PB2: no longer names the net of R15.1, U3.28 (BOOT1/PB2)
- removed net PB6_SCL: R16.2, U3.58 (CAN2_TX/I2C1_SCL/TIM4_CH1/USART1_TX/PB6), U4.6 (SCL)
- removed net PB7_SDA: R17.2, U3.59 (I2C1_SDA/TIM4_CH2/USART1_RX/PB7), U4.7 (SDA)
- new net: C28.1, D5.6
- new net PA8: P1.13 (P13), U3.41 (I2C3_SCL/RCC_MCO_1/TIM1_CH1/USART1_CK/USB_OTG_FS_SOF/PA8)
- new net PB6: P2.13 (P13), U3.58 (CAN2_TX/I2C1_SCL/TIM4_CH1/USART1_TX/PB6)
- new net PB7: P2.12 (P12), U3.59 (I2C1_SDA/TIM4_CH2/USART1_RX/PB7)
- new net PC6: P1.11 (P11), U3.37 (PC6/I2S2_MCK/SDIO_D6/TIM3_CH1/TIM8_CH1/USART6_TX)
- new net PC7: P1.12 (P12), U3.38 (PC7/I2S3_MCK/SDIO_D7/TIM3_CH2/TIM8_CH2/USART6_RX)
- no-connect marks 20 -> 21
Other:
- moved on the sheet: C14, C23, C26, C27, D4, J1, R12, R13, R15, R16, R17, SW2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

Commit message: completed connect tracks
Parts:
- removed C5: 100nF, lib:C_0603, symbol C_Small
- X1: footprint lib:Crystal_SMD_3225_4Pads -> lib:Crystal_SMD_5032_4Pads
