File: gsm-iot-core.kicad_pcb (KiCad board)
At the start: 2 copper layers, 44.7 x 67.6 mm, 99 parts, among them J1 MICRO_SD_HINGE - Micro SD soc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, P1 CONN_01X02, P2 CONN_01X04, P3 CONN_01X15, P4 CONN_01X17, P5 Chip anten, P8 CONN_01X01, Q1 2SC1815, Q2 2SC1815, SW3 SW_PUSH, U1 MP2365DN, U2 LP2985-50DBVR, U3 STM32F405RGTx, U4 MMA7660, U5 SIM800C, U6 SIM HOLD - PPSS-6P, X1 CRYSTAL-24M, Y3 32.768MHz

Commit message: Branch LONGER
Parts:
- C1, C2, C3, C4, C5, C6, C7: footprint Capacitors_SMD:C_0603 -> lib:C_0603
- C29: moved to F.Cu
- J1: footprint MicroSD_Push-Push-A -> lib:MicroSD_Push-Push-A; moved to B.Cu
- U3: footprint TQFP-64_10x10mm_Pitch0.5mm -> lib:TQFP-64_10x10mm_Pitch0.5mm
- U6: footprint SIM_HOLD_115A-ADA0-R02 -> lib:SIM_HOLD_115A-ADA0-R02
- moved R12 42.9 mm to (122.7, 139.7)
- moved R10 41.6 mm to (118.6, 137.2)
- moved R16 39.8 mm to (168.3, 122.5)
- moved C28 39.8 mm to (168.4, 123.7)
- moved SW3 39.8 mm to (168.4, 125.9)
- moved C14 38.5 mm to (154.0, 123.6)
- moved RST 38.5 mm to (154.0, 125.8)
- moved R8 38.5 mm to (154.0, 122.3)
- moved R24 37.0 mm to (190.5, 75.4)
- moved D6 36.8 mm to (189.6, 70.5)
- moved C36 36.5 mm to (190.5, 79.5)
- moved R21 33.6 mm to (200.7, 139.7)
- moved C17 32.4 mm to (128.7, 139.7)
- moved U4 31.8 mm to (200.0, 134.2)
- moved R23 31.7 mm to (187.2, 73.7)
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Connections:
- U4 pad 11: GND -> Net-(U4-Pad11)
Routing:
- net GND: track 409.3 -> 5.14 mm, vias 17 -> 0
- net +3V3: track 252.0 -> 0.00 mm, vias 15 -> 0
- net VDD: track 117.7 -> 0.00 mm, vias 5 -> 0
- net SIM800C_DATA: track 65.4 -> 0.00 mm, vias 4 -> 0
- net /PB2: track 54.5 -> 0.00 mm, vias 5 -> 0
- net PA7_PWRKEY: track 45.6 -> 0.00 mm, vias 4 -> 0
- net +5V: track 42.2 -> 0.00 mm, vias 2 -> 0
- net /PB5: track 36.1 -> 0.00 mm, vias 1 -> 0
- net SIM800C_TXD: track 33.5 -> 0.00 mm, vias 2 -> 0
- net PB3_BUTTON: track 32.2 -> 0.00 mm, vias 2 -> 0
- net SIM800C_RXD: track 31.5 -> 0.00 mm, vias 2 -> 0
- net Net-(C21-Pad1): track 30.1 -> 0.00 mm, vias 2 -> 0
- net /RST: track 27.7 -> 0.00 mm, vias 2 -> 0
- net SIM800C_RST: track 27.3 -> 0.00 mm, vias 1 -> 0
- net SIM800C_VDD: track 27.0 -> 0.00 mm, vias 1 -> 0
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- removed copper zone on B.Cu, net GND
- removed copper zone on F.Cu, net GND
Other:
- board size 44.7 x 67.6 mm -> 25.4 x 86.4 mm
- board text removed: "3.3V"
- board text removed: "5V"
- board text removed: "GND"
- board text removed: "PA0"
- board text removed: "PA1"
- board text removed: "PA2"
- board text removed: "PA3"
- board text removed: "PA4"
- board text removed: "PA5"
- board text removed: "PA6"
- board text removed: "PB1"
- board text removed: "PB10"
- board text removed: "PB11"
- board text removed: "PB12"
- board text removed: "PB13"
- board text removed: "PB14"
- board text removed: "PC0"
- board text removed: "PC1"
- board text removed: "PC13"
- board text removed: "PC2"
- board text removed: "PC3"
- board text removed: "PC4"
- board text removed: "PC8"
- board text removed: "PC9"
- board text removed: "SWCLK"
- board text removed: "SWDIO"
- board text removed: "VBAT"

Commit message: Fails
Parts:
- R14: moved to B.Cu
- moved R12 50.2 mm to (161.2, 107.5), turned to 270 degrees
- moved R10 49.9 mm to (158.7, 107.5), turned to 90 degrees
- moved C21 44.3 mm to (161.2, 115.2), turned to 180 degrees
- moved C17 43.1 mm to (157.4, 107.5), turned to 90 degrees
- moved C6 39.2 mm to (158.8, 117.6), turned to 180 degrees
- moved R11 37.7 mm to (162.6, 107.5), turned to 90 degrees
- moved C24 37.6 mm to (165.1, 107.4), turned to 90 degrees
- moved C18 37.5 mm to (167.7, 116.3), turned to 180 degrees
- moved C1 37.4 mm to (158.8, 116.3), turned to 180 degrees
- moved C20 36.9 mm to (159.9, 107.5), turned to 90 degrees
- moved C22 36.6 mm to (163.9, 107.4), turned to 90 degrees
- moved C5 35.6 mm to (158.8, 115.0), turned to 180 degrees
- moved R9 35.5 mm to (167.7, 115.0), turned to 0 degrees
- moved R20 34.7 mm to (167.7, 113.6), turned to 0 degrees
- moved R18 34.0 mm to (167.7, 112.3), turned to 0 degrees
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Connections:
- U4 pad 11: Net-(U4-Pad11) -> GND
Routing:
- net GND: track 5.14 -> 261.1 mm, vias 0 -> 18
- net +3V3: track 0.00 -> 167.1 mm, vias 0 -> 10
- net /PB2: track 0.00 -> 69.0 mm, vias 0 -> 3
- net +5V: track 0.00 -> 56.1 mm, vias 0 -> 2
- net PA7_PWRKEY: track 0.00 -> 39.6 mm, vias 0 -> 2
- net VDD: track 0.00 -> 37.8 mm, vias 0 -> 1
- net PA10_ID: track 0.00 -> 30.9 mm, vias 0 -> 2
- net PA9_VBUS: track 0.00 -> 29.9 mm
- net PA11_DM: track 0.00 -> 29.8 mm
- net PA12_DP: track 0.00 -> 29.4 mm
- net /PB5: track 0.00 -> 28.5 mm, vias 0 -> 1
- net SIM800C_PWRKEY: track 0.00 -> 25.1 mm
- net SIM800C_RI: track 0.00 -> 25.1 mm, vias 0 -> 2
- net SIM800C_DTR: track 0.00 -> 23.2 mm, vias 0 -> 2
- net PA14_SWCLK: track 0.00 -> 22.1 mm, vias 0 -> 2
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
Commit message: fix PCB
Parts:
- removed P4: CONN_01X17, Pin_Headers:Pin_Header_Straight_1x17
- removed P8 (x4): CONN_01X01, lib:MountingHole_2.5mm
- removed R19, R21: 10k, lib:R_0603
- removed RST: SW_PUSH, lib:SW_SPST_B3U-1000P-B
- added R1: 10K, lib:R_0603, B.Cu at (169.4, 94.0)
- added SW1: SW_PUSH, lib:SW_SPST_B3U-1000P-B, F.Cu at (152.2, 124.4)
- C1, C10, C11, C12, C13, C15, C2, C23, C3, C37, C38, C4, C5, C6, C7, C8, R18, R20, R9, U3, X1, Y3: moved to B.Cu
- C17, C20, C21, C22, C24, C25, C26, C35, C36, D3, D6, L1, R10, R11, R12, R22, R23, R24, U1, U2: moved to F.Cu
- P1: value CONN_01X02 -> CONN_01X16; footprint Pin_Headers:Pin_Header_Straight_1x02 -> Pin_Headers:Pin_Header_Straight_1x16
- P3: value CONN_01X15 -> CONN_01X16; footprint Pin_Headers:Pin_Header_Straight_1x15 -> Pin_Headers:Pin_Header_Straight_1x16
- U6: footprint lib:SIM_HOLD_115A-ADA0-R02 -> lib:115I-AEAA
- moved P1 46.6 mm to (149.9, 76.2), turned to 0 degrees
- moved C25 39.7 mm to (158.7, 93.3), turned to 90 degrees
- moved U2 37.8 mm to (161.3, 93.3), turned to 0 degrees
- moved C26 36.1 mm to (163.9, 93.3), turned to 270 degrees
- moved P2 35.8 mm to (141.1, 84.1), turned to 0 degrees
- moved C18 34.6 mm to (140.3, 95.1)
- moved C6 33.7 mm to (165.1, 84.4), turned to 90 degrees
- moved C1 32.2 mm to (163.8, 84.4), turned to 90 degrees
- moved C35 31.0 mm to (166.4, 67.7), turned to 180 degrees
- moved R23 31.0 mm to (166.4, 66.4), turned to 0 degrees
- moved C5 30.8 mm to (162.5, 84.4), turned to 90 degrees
- moved C7 29.4 mm to (161.2, 84.4), turned to 90 degrees
- moved C3 28.1 mm to (160.0, 84.4), turned to 90 degrees
- moved C2 26.9 mm to (158.8, 84.4), turned to 90 degrees
- moved C8 25.9 mm to (152.6, 108.1), turned to 180 degrees
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Connections:
- C27 pad 1: /PB5 -> +3V3
- P1 pad 1: +5V -> VBAT
- P1 pad 2: VBAT -> +3V3
- P3 pad 10: PC13 -> PB11
- P3 pad 11: PB9 -> PB12
- P3 pad 12: PB8 -> PB13
- P3 pad 13: PB4 -> PB14
- P3 pad 14: GND -> PB15
- P3 pad 2: +3V3 -> GND
- P3 pad 3: GND -> PA3
- P3 pad 4: PA1 -> PA4
- P3 pad 5: PA0 -> PA5
- P3 pad 6: PC3 -> PA6
- P3 pad 7: PC2 -> PB1
- P3 pad 8: PC1 -> PB2
- P3 pad 9: PC0 -> PB10
- U3 pad 28: /PB2 -> PB2
- U3 pad 57: /PB5 -> PB5
- U4 pad 3: /PB5 -> +3V3
- U4 pad 5: /PB2 -> PB5
Routing:
- net GND: track 261.1 -> 3.24 mm, vias 18 -> 0
- net +3V3: track 167.1 -> 1.64 mm, vias 10 -> 0
- net /PB2: track 69.0 -> 0.00 mm, vias 3 -> 0
- net +5V: track 56.1 -> 0.00 mm, vias 2 -> 0
- net PA7_PWRKEY: track 39.6 -> 0.00 mm, vias 2 -> 0
- net VDD: track 37.8 -> 0.00 mm, vias 1 -> 0
- net PA10_ID: track 30.9 -> 0.00 mm, vias 2 -> 0
- net PA9_VBUS: track 29.9 -> 0.00 mm
- net PA11_DM: track 29.8 -> 0.00 mm
- net PA12_DP: track 29.4 -> 0.00 mm
- net /PB5: track 28.5 -> 0.00 mm, vias 1 -> 0
- net SIM800C_PWRKEY: track 25.1 -> 0.00 mm
- net SIM800C_RI: track 25.1 -> 0.00 mm, vias 2 -> 0
- net SIM800C_DTR: track 23.2 -> 0.00 mm, vias 2 -> 0
- net PA14_SWCLK: track 22.1 -> 0.00 mm, vias 2 -> 0
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Other:
- board size 25.4 x 86.4 mm -> 25.4 x 61 mm

Commit message: Fail
Parts:
- C18: moved to B.Cu
- moved P2 56.6 mm to (185.1, 119.7), turned to 180 degrees
- moved C21 50.1 mm to (189.8, 98.6), turned to 90 degrees
- moved R10 48.2 mm to (188.6, 98.6), turned to 90 degrees
- moved R12 46.9 mm to (187.3, 98.6), turned to 90 degrees
- moved C24 46.3 mm to (186.6, 101.9)
- moved C22 46.3 mm to (186.6, 100.7)
- moved R11 45.7 mm to (186.0, 98.6), turned to 270 degrees
- moved D7 45.0 mm to (186.2, 106.9), turned to 0 degrees
- moved C20 44.2 mm to (184.6, 98.6), turned to 270 degrees
- moved C17 43.1 mm to (183.4, 98.6), turned to 270 degrees
- moved D3 32.5 mm to (198.3, 105.0)
- moved L1 26.0 mm to (181.1, 104.9)
- moved Q2 25.5 mm to (197.9, 69.3)
- moved R30 25.5 mm to (197.2, 72.3)
- moved R32 25.5 mm to (198.6, 72.3)
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Routing:
- net PA9_VBUS: track 0.00 -> 23.6 mm, vias 0 -> 1
- net PA10_ID: track 0.00 -> 19.4 mm, vias 0 -> 1
- net PA11_DM: track 0.00 -> 19.2 mm, vias 0 -> 1
- net PB5: track 0.00 -> 19.1 mm
- net PA0: track 16.0 -> 0.00 mm, vias 1 -> 0
- net PC8_SDIO_D0: track 0.00 -> 15.8 mm
- net PA2: track 15.6 -> 0.00 mm
- net PA12_DP: track 0.00 -> 15.3 mm, vias 0 -> 1
- net PA3: track 15.3 -> 0.00 mm
- net PA1: track 15.3 -> 0.00 mm
- net PC3: track 13.9 -> 0.00 mm, vias 1 -> 0
- net PC9_SDIO_D1: track 0.00 -> 13.9 mm, vias 0 -> 1
- net PA4: track 13.3 -> 0.00 mm
- net PC2: track 13.0 -> 0.00 mm, vias 1 -> 0
- net PC0: track 13.0 -> 0.00 mm, vias 1 -> 0
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
Commit message: Merge form longer branch
Parts:
- moved D3 12.1 mm to (200.2, 93.0)
Routing:
- net PC8_SDIO_D0: track 15.8 -> 0.00 mm
- net (no net): track 0.00 -> 15.8 mm
Changed lines of the file:
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@@
   (general
     (links 252)
-    (no_connects 133)
-    (area 136.1333 39.04 201.410843 139.196905)
+    (no_connects 237)
+    (area 136.1333 39.04 201.636301 139.196905)
     (thickness 1.6)
     (drawings 10)
-    (tracks 520)
+    (tracks 88)
     (zones 0)
     (modules 93)
@@
   )
   (module lib:do214ab (layer F.Cu)
-    (at 198.3486 105.0036 270)
+    (at 200.2028 93.03512 270)
     (descr DO214AB)
     (fp_text reference D3 (at 0.03048 3.8227 270) (layer F.SilkS)
@@
     (arrow2b (pts (xy 149.86 58.42) (xy 150.986504 57.833579)))
   )
+  (segment (start 167.5638 103.4796) (end 170.18 106.0958) (width 0.3) (layer F.Cu) (net 0))
+  (segment (start 170.18 106.0958) (end 170.18 113.1062) (width 0.3) (layer F.Cu) (net 0))
+  (segment (start 168.3766 114.9096) (end 165.989004 114.9096) (width 0.3) (layer F.Cu) (net 0))
+  (segment (start 170.18 113.1062) (end 168.3766 114.9096) (width 0.3) (layer F.Cu) (net 0))
+  (segment (start 165.989004 114.9096) (end 165.862004 114.7826) (width 0.3) (layer F.Cu) (net 0))
   (segment (start 164.7571 113.0935) (end 164.7571 111.7629) (width 0.3) (layer B.Cu) (net 2))
   (segment (start 164.7571 111.7629) (end 164.76 111.76) (width 0.3) (layer B.Cu) (net 2))
@@
   (via (at 164.7571 113.0935) (size 1.1) (drill 0.6) (layers F.Cu B.Cu) (net 2))
   (via (at 167.0493 109.4463) (size 1.1) (drill 0.6) (layers F.Cu B.Cu) (net 2))
-  (segment (start 167.5638 103.4796) (end 170.18 106.0958) (width 0.3) (layer F.Cu) (net 23))
-  (segment (start 170.18 106.0958) (end 170.18 113.1062) (width 0.3) (layer F.Cu) (net 23))
-  (segment (start 168.3766 114.9096) (end 165.989004 114.9096) (width 0.3) (layer F.Cu) (net 23))
-  (segment (start 170.18 113.1062) (end 168.3766 114.9096) (width 0.3) (layer F.Cu) (net 23))
-  (segment (start 165.989004 114.9096) (end 165.862004 114.7826) (width 0.3) (layer F.Cu) (net 23))
   (segment (start 167.719317 113.919) (end 166.9415 113.919) (width 0.3) (layer F.Cu) (net 24))
   (segment (start 169.5069 112.9157) (end 168.5036 113.919) (width 0.3) (layer F.Cu) (net 24))
